File: schematics/atmega-dcf77-clock/atmega-dcf77-clock.kicad_pcb (KiCad board)
At the start: 2 copper layers, 70 x 45 mm, 25 parts, among them J1 Barrel_Jack, J2 LCD Module, J3 DCF77, J4 ICSP, SW1 SW_LIGHT, SW2 SW_RESET, U1 MAX667, U2 ATmega324PA-PU

Commit message: Fixed PCB/small fixes
Parts:
- J3: value DCF77 -> DCF77 Receiver Module
- J4: value ICSP -> Conn_02x03_Odd_Even
Connections:
- U2 pad 14: Net-(J2-Pad9) -> (no net)
- U2 pad 15: (no net) -> Net-(J2-Pad9)
Routing:
- net Net-(J2-Pad9): track 15.6 -> 16.7 mm
Changed lines of the file:
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@@
   )
   (setup
-    (last_trace_width 1)
+    (last_trace_width 0.25)
     (user_trace_width 1)
     (trace_clearance 0.2)
@@
     (pad 13 thru_hole oval (at 0 30.48 270) (size 1.6 1.6) (drill 0.8) (layers *.Cu *.Mask))
     (pad 33 thru_hole oval (at 15.24 17.78 270) (size 1.6 1.6) (drill 0.8) (layers *.Cu *.Mask))
-    (pad 14 thru_hole oval (at 0 33.02 270) (size 1.6 1.6) (drill 0.8) (layers *.Cu *.Mask)
+    (pad 14 thru_hole oval (at 0 33.02 270) (size 1.6 1.6) (drill 0.8) (layers *.Cu *.Mask))
+    (pad 34 thru_hole oval (at 15.24 15.24 270) (size 1.6 1.6) (drill 0.8) (layers *.Cu *.Mask))
+    (pad 15 thru_hole oval (at 0 35.56 270) (size 1.6 1.6) (drill 0.8) (layers *.Cu *.Mask)
       (net 6 "Net-(J2-Pad9)"))
-    (pad 34 thru_hole oval (at 15.24 15.24 270) (size 1.6 1.6) (drill 0.8) (layers *.Cu *.Mask))
-    (pad 15 thru_hole oval (at 0 35.56 270) (size 1.6 1.6) (drill 0.8) (layers *.Cu *.Mask))
     (pad 35 thru_hole oval (at 15.24 12.7 270) (size 1.6 1.6) (drill 0.8) (layers *.Cu *.Mask))
     (pad 16 thru_hole oval (at 0 38.1 270) (size 1.6 1.6) (drill 0.8) (layers *.Cu *.Mask))
@@
       (effects (font (size 1 1) (thickness 0.15)))
     )
-    (fp_text value ICSP (at 2.79 2.28 90) (layer F.Fab)
+    (fp_text value Conn_02x03_Odd_Even (at 2.79 2.28 90) (layer F.Fab)
       (effects (font (size 1 1) (thickness 0.15)))
     )
@@
       (effects (font (size 1 1) (thickness 0.15)))
     )
-    (fp_text value DCF77 (at 0.15 2.15 90) (layer F.Fab)
+    (fp_text value "DCF77 Receiver Module" (at 0.15 2.15 90) (layer F.Fab)
       (effects (font (size 1 1) (thickness 0.15)))
     )
@@
   (segment (start 50.2 92.3) (end 52.6 92.3) (width 1) (layer F.Cu) (net 5))
   (segment (start 52.6 92.3) (end 55.3 89.6) (width 1) (layer F.Cu) (net 5))
-  (segment (start 70.53 98.6) (end 73.6 95.53) (width 0.25) (layer B.Cu) (net 6))
   (segment (start 73.6 88.56) (end 76.66 85.5) (width 0.25) (layer B.Cu) (net 6))
-  (segment (start 73.6 95.53) (end 73.6 88.56) (width 0.25) (layer B.Cu) (net 6))
+  (segment (start 67.99 98.6) (end 73.6 92.99) (width 0.25) (layer B.Cu) (net 6))
+  (segment (start 73.6 92.99) (end 73.6 88.56) (width 0.25) (layer B.Cu) (net 6))
   (segment (start 103.695001 98.399997) (end 103.695001 99.190001) (width 0.25) (layer B.Cu) (net 7))
   (segment (start 42.8 111.76) (end 45.94 114.9) (width 0.25) (layer F.Cu) (net 7))
